File: electronics/PCB/project-files/thermometer-digital-min_max-pcb/thermometer-digital-min_max-pcb.kicad_sch (KiCad schematic)
At the start: 29 parts, among them J0 sensor_connection, J1 battery_connection, Q0 PN2222A, Q1 PN2222A, Q2 PN2222A, Q3 PN2222A, U0 ATmega328P-U

Commit message: Testing signing
Connections:
- net GND: now also U0.10 (XTAL2/PB7), U0.19 (PB5), U0.20 (AVCC), U0.21 (AREF), U0.27 (PC4), U0.28 (PC5), U0.9 (XTAL1/PB6)
Changed lines of the file:
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@@
     (rev "1")
   )
+  (junction (at 100.33 81.28) (diameter 0) (color 0 0 0 0)
+  )
   (junction (at 48.26 45.72) (diameter 0) (color 0 0 0 0)
   )
@@
   (junction (at 205.74 83.82) (diameter 0) (color 0 0 0 0)
   )
+  (junction (at 100.33 101.6) (diameter 0) (color 0 0 0 0)
+  )
   (junction (at 38.1 50.8) (diameter 0) (color 0 0 0 0)
   )
@@
     (stroke (width 0) (type default) (color 0 0 0 0))
   )
+  (wire (pts (xy 93.98 53.34) (xy 93.98 54.61))
+    (stroke (width 0) (type default) (color 0 0 0 0))
+  )
   (wire (pts (xy 149.86 54.61) (xy 149.86 68.58))
     (stroke (width 0) (type default) (color 0 0 0 0))
@@
     (stroke (width 0) (type default) (color 0 0 0 0))
   )
+  (wire (pts (xy 105.41 81.28) (xy 105.41 82.55))
+    (stroke (width 0) (type default) (color 0 0 0 0))
+  )
   (wire (pts (xy 116.84 128.27) (xy 123.19 128.27))
     (stroke (width 0) (type default) (color 0 0 0 0))
@@
     (stroke (width 0) (type default) (color 0 0 0 0))
   )
+  (wire (pts (xy 67.31 66.04) (xy 67.31 67.31))
+    (stroke (width 0) (type default) (color 0 0 0 0))
+  )
   (bus (pts (xy 173.99 52.07) (xy 175.26 52.07))
     (stroke (width 0) (type default) (color 0 0 0 0))
@@
     (stroke (width 0) (type default) (color 0 0 0 0))
   )
+  (wire (pts (xy 100.33 101.6) (xy 130.81 101.6))
+    (stroke (width 0) (type default) (color 0 0 0 0))
+  )
   (wire (pts (xy 85.09 40.64) (xy 113.03 40.64))
     (stroke (width 0) (type default) (color 0 0 0 0))
@@
     (stroke (width 0) (type default) (color 0 0 0 0))
   )
+  (wire (pts (xy 69.85 66.04) (xy 67.31 66.04))
+    (stroke (width 0) (type default) (color 0 0 0 0))
+  )
   (wire (pts (xy 250.19 54.61) (xy 250.19 66.04))
     (stroke (width 0) (type default) (color 0 0 0 0))
@@
     (stroke (width 0) (type default) (color 0 0 0 0))
   )
+  (wire (pts (xy 87.63 58.42) (xy 87.63 53.34))
+    (stroke (width 0) (type default) (color 0 0 0 0))
+  )
   (bus (pts (xy 125.73 119.38) (xy 125.73 125.73))
     (stroke (width 0) (type default) (color 0 0 0 0))
@@
     (stroke (width 0) (type default) (color 0 0 0 0))
   )
+  (wire (pts (xy 100.33 81.28) (xy 100.33 83.82))
+    (stroke (width 0) (type default) (color 0 0 0 0))
+  )
   (wire (pts (xy 172.72 81.28) (xy 172.72 83.82))
     (stroke (width 0) (type default) (color 0 0 0 0))
@@
     (stroke (width 0) (type default) (color 0 0 0 0))
   )
+  (wire (pts (xy 100.33 81.28) (xy 105.41 81.28))
+    (stroke (width 0) (type default) (color 0 0 0 0))
+  )
   (wire (pts (xy 33.02 43.18) (xy 38.1 43.18))
     (stroke (width 0) (type default) (color 0 0 0 0))
@@
     (stroke (width 0) (type default) (color 0 0 0 0))
   )
+  (wire (pts (xy 87.63 53.34) (xy 93.98 53.34))
+    (stroke (width 0) (type default) (color 0 0 0 0))
+  )
   (bus (pts (xy 172.72 52.07) (xy 173.99 52.07))
     (stroke (width 0) (type default) (color 0 0 0 0))
@@
     (stroke (width 0) (type default) (color 0 0 0 0))
   )
+  (wire (pts (xy 100.33 99.06) (xy 100.33 101.6))
+    (stroke (width 0) (type default) (color 0 0 0 0))
+  )
   (wire (pts (xy 212.09 76.2) (xy 212.09 54.61))
     (stroke (width 0) (type default) (color 0 0 0 0))
@@
     (stroke (width 0) (type default) (color 0 0 0 0))
   )
+  (wire (pts (xy 130.81 101.6) (xy 130.81 109.22))
+    (stroke (width 0) (type default) (color 0 0 0 0))
+  )
   (wire (pts (xy 179.07 76.2) (xy 189.23 76.2))
     (stroke (width 0) (type default) (color 0 0 0 0))
   )
   (wire (pts (xy 118.11 30.48) (xy 119.38 30.48))
+    (stroke (width 0) (type default) (color 0 0 0 0))
+  )
+  (wire (pts (xy 100.33 78.74) (xy 100.33 81.28))
     (stroke (width 0) (type default) (color 0 0 0 0))
   )
@@
     )
     (property "Datasheet" "" (id 3) (at 271.78 139.7 0)
+      (effects (font (size 1.27 1.27)) hide)
+    )
+    (pin "1")
+  )
+  (symbol (lib_id "power:GND") (at 130.81 109.22 0) (unit 1)
+    (in_bom yes) (on_board yes) (fields_autoplaced)
+    (property "Reference" "#PWR?" (id 0) (at 130.81 115.57 0)
+      (effects (font (size 1.27 1.27)) hide)
+    )
+    (property "Value" "GND" (id 1) (at 130.81 114.3 0))
+    (property "Footprint" "" (id 2) (at 130.81 109.22 0)
+      (effects (font (size 1.27 1.27)) hide)
+    )
+    (property "Datasheet" "" (id 3) (at 130.81 109.22 0)
       (effects (font (size 1.27 1.27)) hide)
     )
@@
     (pin "9")
   )
+  (symbol (lib_id "power:GND") (at 105.41 82.55 0) (unit 1)
+    (in_bom yes) (on_board yes) (fields_autoplaced)
+    (property "Reference" "#PWR?" (id 0) (at 105.41 88.9 0)
+      (effects (font (size 1.27 1.27)) hide)
+    )
+    (property "Value" "GND" (id 1) (at 105.41 87.63 0))
+    (property "Footprint" "" (id 2) (at 105.41 82.55 0)
+      (effects (font (size 1.27 1.27)) hide)
+    )
+    (property "Datasheet" "" (id 3) (at 105.41 82.55 0)
+      (effects (font (size 1.27 1.27)) hide)
+    )
+    (pin "1")
+  )
   (symbol (lib_id "power:VCC") (at 38.1 35.56 0) (unit 1)
     (in_bom yes) (on_board yes) (fields_autoplaced)
@@
     (pin "1")
     (pin "2")
+  )
+  (symbol (lib_id "power:GND") (at 67.31 67.31 0) (unit 1)
+    (in_bom yes) (on_board yes) (fields_autoplaced)
+    (property "Reference" "#PWR?" (id 0) (at 67.31 73.66 0)
+      (effects (font (size 1.27 1.27)) hide)
+    )
+    (property "Value" "GND" (id 1) (at 67.31 72.39 0))
+    (property "Footprint" "" (id 2) (at 67.31 67.31 0)
+      (effects (font (size 1.27 1.27)) hide)
+    )
+    (property "Datasheet" "" (id 3) (at 67.31 67.31 0)
+      (effects (font (size 1.27 1.27)) hide)
+    )
+    (pin "1")
   )
   (symbol (lib_id "power:GND") (at 238.76 127 0) (unit 1)
@@
     (pin "1")
     (pin "2")
+  )
+  (symbol (lib_id "power:GND") (at 93.98 54.61 0) (unit 1)
+    (in_bom yes) (on_board yes) (fields_autoplaced)
+    (property "Reference" "#PWR?" (id 0) (at 93.98 60.96 0)
+      (effects (font (size 1.27 1.27)) hide)
+    )
+    (property "Value" "GND" (id 1) (at 93.98 59.69 0))
+    (property "Footprint" "" (id 2) (at 93.98 54.61 0)
+      (effects (font (size 1.27 1.27)) hide)
+    )
+    (property "Datasheet" "" (id 3) (at 93.98 54.61 0)
+      (effects (font (size 1.27 1.27)) hide)
+    )
+    (pin "1")
   )
   (symbol (lib_id "Device:R") (at 113.03 115.57 90) (unit 1)
@@
       (reference "#PWR0116") (unit 1) (value "VCC") (footprint "")
     )
+    (path "/61220fbd-67c5-4696-a5f7-9d56c7a117fb"
+      (reference "#PWR?") (unit 1) (value "GND") (footprint "")
+    )
+    (path "/a48cb493-8f10-424f-ae52-94cae8da6111"
+      (reference "#PWR?") (unit 1) (value "GND") (footprint "")
+    )
+    (path "/b05fbadb-d42d-49c6-8459-ce3779d5ec39"
+      (reference "#PWR?") (unit 1) (value "GND") (footprint "")
+    )
+    (path "/c89eefab-ae73-493b-93c2-6a70734bd602"
+      (reference "#PWR?") (unit 1) (value "GND") (footprint "")
+    )
     (path "/008e62dc-8141-4dcb-b386-ca39e7f3ce96"
