File: electronics/PCB/project-files/thermometer-digital-min_max-pcb/thermometer-digital-min_max-pcb.kicad_pcb (KiCad board)
At the start: 2 copper layers, 100 x 75 mm, 33 parts, among them J0 sensor_connection, J1 battery_connection, Q0 PN2222A, Q1 PN2222A, Q2 PN2222A, Q3 PN2222A, U0 ATmega328P-U

Commit message: Updated PCB to v1.1
Other:
- board text added: "V1.1"
- board text removed: "V1.0"
Changed lines of the file:
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@@
   (gr_line (start 197 115) (end 107 115) (layer "Edge.Cuts") (width 0.1))
   (gr_line (start 107 40) (end 197 40) (layer "Edge.Cuts") (width 0.1))
-  (gr_text "V1.0" (at 112 110) (layer "F.SilkS")
+  (gr_text "V1.1" (at 112 110) (layer "F.SilkS")
     (effects (font (size 1 1) (thickness 0.15)))
   )
